File: pcb/Lucas11-Dev-Board.kicad_pcb (KiCad board)
At the start: 2 copper layers, 11 parts, among them J1 Conn_01x04, SW3 SW_Push, SW4 SW_Push, SW5 SW_Push, SW6 SW_Push, U1 XIAO-RP2350-SMD

Commit message: Logo wasent centered XD
Parts:
- moved G*** 2.38 mm to (94.9, 47.6)
Changed lines of the file:
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@@
 	(footprint "LOGO"
 		(layer "F.Cu")
-		(at 94.86 45.24375)
+		(at 94.86 47.625)
 		(property "Reference" "G***"
 			(at 0 0 0)

Commit message: Finished the PCB!!!!
Parts:
- moved G*** 0.39 mm to (95.2, 47.6)
Routing:
- net +5V: track 0.00 -> 217.7 mm
- net Net-(D1-DIN): track 0.00 -> 95.6 mm
- net Net-(J1-Pin_4): track 0.00 -> 92.7 mm
- net Net-(J1-Pin_3): track 0.00 -> 92.3 mm
- net Net-(J1-Pin_2): track 0.00 -> 85.5 mm
- net Net-(J1-Pin_1): track 1.03 -> 76.4 mm
- net Net-(D1-DOUT): track 1.03 -> 76.1 mm
- net Net-(U1-GPIO11/D15/SPI1_MOSI): track 0.00 -> 65.3 mm
- net Net-(U1-GPIO12/D16/SPI1_MISO): track 0.00 -> 39.0 mm
- net Net-(U1-GPIO10/D17/SPI1_SCK): track 0.00 -> 37.7 mm
- net Net-(U1-GPIO9/D18/SPI1_CS): track 0.00 -> 32.1 mm
Other:
- board outline added: 81 x 61.9 mm

Commit message: Fix all the DRC errors
Routing:
- net +5V: track 217.7 -> 235.7 mm
- net Net-(J1-Pin_3): track 92.3 -> 103.4 mm
- net Net-(J1-Pin_1): track 76.4 -> 82.7 mm
- net Net-(J1-Pin_2): track 85.5 -> 90.7 mm

Commit message: a
Parts:
- removed U1: XIAO-RP2350-SMD, OPL:XIAO-RP2350-SMD
- added U2: XIAO-RP2350-DIP, OPL:XIAO-RP2350-DIP, F.Cu at (94.3, 22.2)
Connections:
- D1 pad 2: +5V -> GND
- D2 pad 1: unconnected-(D2-DOUT-Pad1) -> Net-(D2-DOUT)
- D2 pad 2: +5V -> GND
- D3 pad 1: unconnected-(D3-DOUT-Pad1) -> Net-(D3-DOUT)
- D3 pad 2: +5V -> GND
- D3 pad 3: Net-(D1-DOUT) -> Net-(D2-DOUT)
- D4 pad 2: +5V -> GND
- D4 pad 3: Net-(D1-DOUT) -> Net-(D3-DOUT)
- SW3 pad 1: +5V -> GND
- SW4 pad 1: +5V -> GND
- SW5 pad 1: +5V -> GND
- SW6 pad 1: +5V -> GND
Routing:
- net GND: track 0.00 -> 245.2 mm
- net +5V: track 235.7 -> 25.4 mm
- net Net-(D1-DIN): track 95.6 -> 0.00 mm
- net Net-(D1-DOUT): track 76.1 -> 0.00 mm
- net Net-(U2-GPIO3/D10/SPI0_MOSI): track 32.1 -> 105.0 mm
- net Net-(U2-GPIO1/D7/RX0): track 65.3 -> 0.00 mm
- net Net-(U2-GPIO4/D9/SPI_MISO): track 37.7 -> 77.2 mm
- net Net-(J1-Pin_1): track 82.7 -> 108.2 mm
- net Net-(J1-Pin_2): track 90.7 -> 67.9 mm
- net Net-(J1-Pin_3): track 103.4 -> 82.3 mm
- net Net-(U2-GPIO2/D8/SPI0_SCK): track 39.0 -> 21.2 mm
- net Net-(J1-Pin_4): track 92.7 -> 90.4 mm
- net unconnected-(U2-3V3-Pad12): track 0.00 -> 0.65 mm
